File: Kicad/MicroWordClockTut.sch (KiCad schematic (older format))
At the start: 10 parts, among them J1 Conn_01x02_Male, J2 Conn_02x03_Male, SW1 SW_SPST, U1 ATmega328P-AU, U2 8x8_LED_MATRIX, U3 DS1307Z+, U4 8x8_LED_MATRIX, Y1 Crystal

Commit message: started routing.  it is small.  pinswapped a lot
Parts:
- removed J1: Conn_01x02_Male, Connector_PinHeader_2.54mm:PinHeader_1x02_P2.54mm_Vertical, symbol Connector:Conn_01x02_Male
- removed U2: 8x8_LED_MATRIX, MicroWordClockTut:788LEDMATRIX, symbol MicroWordClockTut:8x8_LED_MATRIX
- added BT1: Battery_Cell, MicroWordClockTut:BR1225VCN, symbol Device:Battery_Cell
- added J1: USB_B_Micro, Connectors:USB_Micro-B_10103594-0001LF, symbol Connector:USB_B_Micro
- added R1: 200, Resistors_SMD:R_1206, symbol Device:R
- J2: footprint MicroWordClockTut:2x3 Header -> Connectors:Tag-Connect_TC2030-IDC-NL
Connections:
- net labels added: 1, 10, 12, 13, 14, 2, 23, 24, 25, 26, 30, 31, 32, 7, 8, 9
- net labels removed: C1, C2, C3, C4, C5, C6, C7, C8, R1, R2, R3, R4, R5, R6, R7, R8
- wire segments 85 -> 82
Other:
- note removed: "8X8 LED MATRIX "788""
- moved on the sheet: C1, C2, J2, SW1, U1, U3, U4, Y1

Commit message: latest version with tiny switch NanoT
Parts:
- removed R1: 200, Resistors_SMD:R_1206, symbol Device:R
- removed SW1: SW_SPST, MicroWordClockTut:PTS647 tact switch, symbol MicroWordClockTut:SW_SPST
- added SW1: SW_SPST_2PIN, MicroWordClockTut:NanoT BS, symbol MicroWordClockTut:SW_SPST_2PIN
- J1: footprint Connectors:USB_Micro-B_10103594-0001LF -> MicroWordClockTut:10118192-0001LF
- J2: footprint Connectors:Tag-Connect_TC2030-IDC-NL -> MicroWordClockTut:side connector
Connections:
- wire segments 82 -> 76
Other:
- moved on the sheet: C1
Changed lines of the file:
@@
 L Device:C C1
 U 1 1 601DB948
-P 2900 3950
-F 0 "C1" H 3015 3996 50  0000 L CNN
-F 1 "C" H 3015 3905 50  0000 L CNN
-F 2 "Capacitors_SMD:C_0805_HandSoldering" H 2938 3800 50  0001 C CNN
-F 3 "~" H 2900 3950 50  0001 C CNN
-	1    2900 3950
+P 2950 3950
+F 0 "C1" H 3065 3996 50  0000 L CNN
+F 1 "C" H 3065 3905 50  0000 L CNN
+F 2 "Capacitors_SMD:C_0805_HandSoldering" H 2988 3800 50  0001 C CNN
+F 3 "~" H 2950 3950 50  0001 C CNN
+	1    2950 3950
 	1    0    0    -1
 $EndComp
@@
 L power:GND #PWR02
 U 1 1 601E0DF0
-P 2900 4200
-F 0 "#PWR02" H 2900 3950 50  0001 C CNN
-F 1 "GND" H 2905 4027 50  0000 C CNN
-F 2 "" H 2900 4200 50  0001 C CNN
-F 3 "" H 2900 4200 50  0001 C CNN
-	1    2900 4200
+P 2950 4200
+F 0 "#PWR02" H 2950 3950 50  0001 C CNN
+F 1 "GND" H 2955 4027 50  0000 C CNN
+F 2 "" H 2950 4200 50  0001 C CNN
+F 3 "" H 2950 4200 50  0001 C CNN
+	1    2950 4200
 	1    0    0    -1
 $EndComp
@@
 L power:+5V #PWR01
 U 1 1 601E148A
-P 2900 3650
-F 0 "#PWR01" H 2900 3500 50  0001 C CNN
-F 1 "+5V" H 2915 3823 50  0000 C CNN
-F 2 "" H 2900 3650 50  0001 C CNN
-F 3 "" H 2900 3650 50  0001 C CNN
-	1    2900 3650
-	1    0    0    -1
-$EndComp
-Wire Wire Line
-	2900 3650 2900 3800
+P 2950 3650
+F 0 "#PWR01" H 2950 3500 50  0001 C CNN
+F 1 "+5V" H 2965 3823 50  0000 C CNN
+F 2 "" H 2950 3650 50  0001 C CNN
+F 3 "" H 2950 3650 50  0001 C CNN
+	1    2950 3650
+	1    0    0    -1
+$EndComp
+Wire Wire Line
+	2950 3650 2950 3800
 $Comp
 L power:+5V #PWR03
@@
 	3300 3650 3300 3800
 Wire Wire Line
-	2900 4100 2900 4200
+	2950 4100 2950 4200
 Wire Wire Line
 	3300 4100 3300 4200
@@
 F 0 "J2" H 2600 5650 50  0000 C CNN
 F 1 "Conn_02x03_Male" H 2900 5750 50  0000 C CNN
-F 2 "Connectors:Tag-Connect_TC2030-IDC-NL" H 3150 5400 50  0001 C CNN
+F 2 "MicroWordClockTut:side connector" H 3150 5400 50  0001 C CNN
 F 3 "~" H 3150 5400 50  0001 C CNN
 	1    3150 5300
@@
 Wire Wire Line
 	3350 5300 3700 5300
-Text Label 2550 5100 0    50   ~ 0
+Text Label 3450 5200 0    50   ~ 0
 MISO
 Text Label 2550 5200 0    50   ~ 0
 SCK
+Text Label 2550 5100 0    50   ~ 0
+RST
 Text Label 2550 5300 0    50   ~ 0
-RST
-Text Label 3450 5200 0    50   ~ 0
 MOSI
 $Comp
@@
 Text Notes 7600 3650 0    50   ~ 0
 8X8 LED MATRIX FROM ADAFRUIT
-$Comp
-L MicroWordClockTut:SW_SPST SW1
-U 1 1 6025B2B1
-P 6500 4850
-F 0 "SW1" H 6500 5085 50  0000 C CNN
-F 1 "SW_SPST" H 6500 4994 50  0000 C CNN
-F 2 "MicroWordClockTut:PTS647 tact switch" H 6500 4850 50  0001 C CNN
-F 3 "~" H 6500 4850 50  0001 C CNN
-	1    6500 4850
-	1    0    0    -1
-$EndComp
 Wire Wire Line
 	8800 1800 8800 2100
@@
 F 0 "J1" H 2757 2667 50  0000 C CNN
 F 1 "USB_B_Micro" H 2757 2576 50  0000 C CNN
-F 2 "Connectors:USB_Micro-B_10103594-0001LF" H 2850 2150 50  0001 C CNN
+F 2 "MicroWordClockTut:10118192-0001LF" H 2850 2150 50  0001 C CNN
 F 3 "~" H 2850 2150 50  0001 C CNN
 	1    2700 2200
@@
 Wire Wire Line
 	2650 2650 2700 2650
-$Comp
-L Device:R R1
-U 1 1 60429384
-P 3400 2250
-F 0 "R1" H 3470 2296 50  0000 L CNN
-F 1 "200" H 3470 2205 50  0000 L CNN
-F 2 "Resistors_SMD:R_1206" V 3330 2250 50  0001 C CNN
-F 3 "~" H 3400 2250 50  0001 C CNN
-	1    3400 2250
-	1    0    0    -1
-$EndComp
-Wire Wire Line
-	3000 2200 3150 2200
-Wire Wire Line
-	3150 2200 3150 2100
-Wire Wire Line
-	3150 2100 3400 2100
-Wire Wire Line
-	3000 2300 3150 2300
-Wire Wire Line
-	3150 2300 3150 2400
-Wire Wire Line
-	3150 2400 3400 2400
 $Comp
 L Device:Battery_Cell BT1
@@
 Text Label 9500 5000 0    50   ~ 0
 2
+$Comp
+L MicroWordClockTut:SW_SPST_2PIN SW1
+U 1 1 6044E743
+P 6500 4850
+F 0 "SW1" H 6500 5085 50  0000 C CNN
+F 1 "SW_SPST_2PIN" H 6500 4994 50  0000 C CNN
+F 2 "MicroWordClockTut:NanoT BS" H 6500 4850 50  0001 C CNN
+F 3 "~" H 6500 4850 50  0001 C CNN
+	1    6500 4850
+	1    0    0    -1
+$EndComp
 $EndSCHEMATC
